File: design/programmableAmplifier/programmableAmplifier.kicad_sch (KiCad schematic)
At the start: 11 parts, among them Q2 2N3904, U3 LM324

Commit message: Finished the weight design
Parts:
- added Q1, Q3, Q4: 2N3904, Package_TO_SOT_THT:TO-92_Inline, symbol Transistor_BJT:2N3904
- added R10, R4, R7: 1k, Resistor_SMD:R_0402_1005Metric, symbol Device:R_Small
- added R11, R12, R5, R8: 100k, Resistor_SMD:R_0402_1005Metric, symbol Device:R_Small
- added R6: 3.3k, Resistor_SMD:R_0402_1005Metric, symbol Device:R_Small
- added R9: 10k, Resistor_SMD:R_0402_1005Metric, symbol Device:R_Small
- R3: value 10k -> 1.4k
Connections:
- net +3.3V: no longer R1.1, R2.1
- net 0: now also Q1.1 (E), Q3.1 (E), Q4.1 (E), R11.2, R5.2, R8.2
- net at R19.2, R3.1, U3.2 (-): now also R12.1, R6.1, R9.1
- new net: Q3.3 (C), R9.2
- new net: Q3.2 (B), R7.2
- new net: Q1.2 (B), R4.2
- new net: Q1.3 (C), R6.2
- new net: Q4.3 (C), R12.2
- new net: Q4.2 (B), R10.2
- new net pga_ctrl0: R1.1, R2.1
- new net pga_ctrl1: R4.1, R5.1
- new net pga_ctrl2: R7.1, R8.1
- new net pga_ctrl3: R10.1, R11.1
Other:
- note added: "Simulated amplifiations: 100k = 1.1x 10k = 2x 3k3 = 4x 1k4 = 8x"
- moved on the sheet: Q2, R1, R19, R2, R3
